File: hardware/SCLF_Gripper.kicad_sch (KiCad schematic)
At the start: 73 parts, among them J1 Conn_01x05, J2 Conn_01x03, J3 Coupling_02x05_Odd_Even, Q1 AO3401A, SW1 TSA002A3512A02, SW2 TSA002A3512A02, U1 DRV8316CRRGFR, U10 XC6206P332MR, U4 MAX3485, U8 MT6701QT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

Commit message: docs: update pinout, images to PNG and hardware design files
Parts:
- added C4: 100nF, Capacitor_SMD:C_0402_1005Metric, symbol Device:C
- added F1: Fuse, Fuse:Fuse_1206_3216Metric_Pad1.42x1.75mm_HandSolder, symbol Device:Fuse
- added TP3: VIN, TestPoint:TestPoint_Pad_D1.0mm, symbol Connector:TestPoint
- J2: footprint Connector_PinHeader_2.54mm:PinHeader_1x03_P2.54mm_Vertical -> Aimar:PinHeader_1x03_P2.54mm_Vertical_Center
Connections:
- net 24V: now also J3.4 (Pin_4), F1.1; no longer D5.2 (A2), D6.1 (K)
- net 3V3: now also C4.1
- net AL: now also U9.28 (PB15); no longer U9.26 (PB13)
- net CL: now also U9.26 (PB13); no longer U9.28 (PB15)
- net GND: now also D5.2 (A2), J3.2 (Pin_2), U1.21 (DRVOFF), C4.2
- net VIN: now also L2.2, TP3.1; no longer L2.1
- net at C1.1, D5.1 (A1): now also D6.1 (K), L2.1, F1.2; no longer L2.2
- net DRV_FAULT: now reaches U9.2 (PC13)
- net DRV_FAULT: now also R25.2, U1.22 (nFAULT)
- net PA15: no longer names the net of U9.38 (PA15)
- net PB6: no longer names the net of U9.44 (PB6)
- net PB7: no longer names the net of U9.45 (PB7)
- no-connect marks 16 -> 15
Other:
- note added: "D5 parallel Added F1 fuse Added VIN test pad Switched AL and CL DRVOFF to GND Added GND and 24V to pins 2 and 4 in input connector Connected nFAULT to PC13"
- note added: "Power and external communication"
- note added: "With current sense, step-down converter"
- note removed: "With current sense, step-down convertor"
- moved on the sheet: C1, C13, C2, C23, C25, C26, C27, C28, C29, C3, C30, C31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
